File: files/kicad/biquad/biquad.kicad_sch (KiCad schematic)
At the start: 15 parts, among them U1 TL082, U2 TL082

Commit message: Modified eqns and labels
Parts:
- renumbered VIN to VIN1
Other:
- note added: ".control set controlswait write biquad.raw all .endc"
- note removed: ".control set controlswait write schaltungsentwurf_no1.raw all .endc"
Changed lines of the file:
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@@
 	(generator_version "9.0")
 	(paper "A4")
-	(text ".control\nset controlswait\nwrite schaltungsentwurf_no1.raw all\n.endc"
+	(text ".control\nset controlswait\nwrite biquad.raw all\n.endc"
 		(exclude_from_sim no)
 		(at 138.43 77.724 0)
@@
 		(dnp no)
 		(fields_autoplaced yes)
-		(property "Reference" "VIN"
+		(property "Reference" "VIN1"
 			(at 78.74 105.2801 0)
 			(effects
@@
 			(project ""
 				(path "/c6c07df8-04b2-428a-b6be-e0bc04b23e84"
-					(reference "VIN")
+					(reference "VIN1")
 					(unit 1)
 				)
